File: Schematico/NOI-domotics-schematico.kicad_sch (KiCad schematic)
At the start: 0 parts

Commit message: new parts
Parts:
- added J?: RASPBERRY PI ZERO W, symbol raspberrypi_zerow_uhat-cache:Connector_Generic_Conn_02x20_Odd_Even
- added K?: FINDER-34.51, Relay_THT:Relay_SPDT_Finder_34.51_Vertical, symbol Relay:FINDER-34.51
- added U?: VO615A-4, symbol Isolator:VO615A-4
- added U?: ESP_32, symbol ESP32:ESP_32
Changed lines of the file:
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@@
 (kicad_sch (version 20211123) (generator eeschema)
   (paper "A4")
+  (symbol (lib_id "Isolator:VO615A-4") (at 224.028 61.468 0) (unit 1)
+    (in_bom yes) (on_board yes)
+    (property "Reference" "U?" (id 0) (at 224.282 42.164 0))
+    (property "Value" "VO615A-4" (id 1) (at 224.79 37.846 0))
+    (property "Footprint" "" (id 2) (at 224.028 61.468 0)
+      (effects (font (size 1.27 1.27)) hide)
+    )
+    (property "Datasheet" "http://www.vishay.com/docs/81753/vo615a.pdf" (id 3) (at 225.298 33.782 0)
+      (effects (font (size 1.27 1.27)) hide)
+    )
+    (pin "")
+    (pin "")
+    (pin "")
+    (pin "")
+    (pin "")
+    (pin "")
+    (pin "")
+    (pin "")
+    (pin "")
+    (pin "")
+    (pin "")
+    (pin "")
+    (pin "L")
+    (pin "L")
+    (pin "L")
+    (pin "L")
+    (pin "L")
+    (pin "L")
+    (pin "L")
+    (pin "L")
+    (pin "N")
+    (pin "N")
+    (pin "N")
+    (pin "N")
+    (pin "N")
+    (pin "N")
+    (pin "N")
+    (pin "N")
+  )
+  (symbol (lib_id "raspberrypi_zerow_uhat-cache:Connector_Generic_Conn_02x20_Odd_Even") (at 133.858 82.55 0) (unit 1)
+    (in_bom yes) (on_board yes)
+    (property "Reference" "J?" (id 0) (at 134.112 48.006 0))
+    (property "Value" "RASPBERRY PI ZERO W" (id 1) (at 134.112 50.546 0))
+    (property "Footprint" "" (id 2) (at 133.858 82.55 0)
+      (effects (font (size 1.27 1.27)) hide)
+    )
+    (property "Datasheet" "" (id 3) (at 133.858 82.55 0)
+      (effects (font (size 1.27 1.27)) hide)
+    )
+    (pin "")
+    (pin "1")
+    (pin "10")
+    (pin "11")
+    (pin "12")
+    (pin "13")
+    (pin "14")
+    (pin "15")
+    (pin "16")
+    (pin "17")
+    (pin "18")
+    (pin "19")
+    (pin "2")
+    (pin "20")
+    (pin "21")
+    (pin "22")
+    (pin "23")
+    (pin "24")
+    (pin "25")
+    (pin "26")
+    (pin "27")
+    (pin "28")
+    (pin "29")
+    (pin "3")
+    (pin "30")
+    (pin "31")
+    (pin "32")
+    (pin "33")
+    (pin "34")
+    (pin "35")
+    (pin "36")
+    (pin "37")
+    (pin "38")
+    (pin "39")
+    (pin "4")
+    (pin "40")
+    (pin "5")
+    (pin "6")
+    (pin "7")
+    (pin "8")
+    (pin "9")
+  )
+  (symbol (lib_id "Relay:FINDER-34.51") (at 68.58 73.66 0) (unit 1)
+    (in_bom yes) (on_board yes) (fields_autoplaced)
+    (property "Reference" "K?" (id 0) (at 93.726 44.9579 0)
+      (effects (font (size 1.27 1.27)) (justify left))
+    )
+    (property "Value" "FINDER-34.51" (id 1) (at 93.726 47.4979 0)
+      (effects (font (size 1.27 1.27)) (justify left))
+    )
+    (property "Footprint" "Relay_THT:Relay_SPDT_Finder_34.51_Vertical" (id 2) (at 91.694 39.116 0)
+      (effects (font (size 1.27 1.27)) hide)
+    )
+    (property "Datasheet" "https://gfinder.findernet.com/public/attachments/34/EN/S34USAEN.pdf" (id 3) (at 85.09 42.926 0)
+      (effects (font (size 1.27 1.27)) hide)
+    )
+    (pin "")
+    (pin "")
+    (pin "")
+    (pin "")
+    (pin "")
+    (pin "")
+    (pin "")
+    (pin "")
+    (pin "")
+    (pin "")
+    (pin "")
+    (pin "")
+    (pin "")
+    (pin "")
+    (pin "")
+    (pin "")
+    (pin "")
+    (pin "")
+    (pin "")
+    (pin "")
+    (pin "")
+    (pin "")
+    (pin "")
+    (pin "")
+    (pin "")
+    (pin "")
+    (pin "")
+    (pin "")
+    (pin "")
+    (pin "")
+    (pin "")
+    (pin "")
+    (pin "")
+    (pin "")
+    (pin "")
+    (pin "")
+    (pin "")
+    (pin "")
+    (pin "")
+    (pin "")
+    (pin "")
+    (pin "")
+    (pin "")
+    (pin "")
+    (pin "")
+    (pin "")
+    (pin "")
+    (pin "")
+  )
+  (symbol (lib_id "ESP32:ESP_32") (at 172.466 57.15 0) (unit 1)
+    (in_bom yes) (on_board yes) (fields_autoplaced)
+    (property "Reference" "U?" (id 0) (at 180.086 43.434 0))
+    (property "Value" "ESP_32" (id 1) (at 180.086 45.974 0))
+    (property "Footprint" "" (id 2) (at 172.466 57.15 0)
+      (effects (font (size 1.27 1.27)) hide)
+    )
+    (property "Datasheet" "" (id 3) (at 172.466 57.15 0)
+      (effects (font (size 1.27 1.27)) hide)
+    )
+    (pin "")
+    (pin "1")
+    (pin "1")
+    (pin "1")
+    (pin "1")
+    (pin "1")
+    (pin "1")
+    (pin "1")
+    (pin "1")
+    (pin "1")
+    (pin "1")
+    (pin "1")
+    (pin "1")
+    (pin "1")
+    (pin "1")
+    (pin "1")
+    (pin "1")
+    (pin "1")
+    (pin "1")
+    (pin "1")
+    (pin "1")
+    (pin "1")
+    (pin "1")
+    (pin "1")
+    (pin "1")
+    (pin "1")
+    (pin "1")
+    (pin "1")
+    (pin "1")
+    (pin "1")
+    (pin "1")
+  )
   (sheet_instances
     (path "/" (page "1"))
   )
+  (symbol_instances
+    (path "/235f4f81-3283-4817-a1ad-c039c7cf2ada"
+      (reference "J?") (unit 1) (value "RASPBERRY PI ZERO W") (footprint "")
+    )
+    (path "/acb6c3f3-e677-4f35-9fc2-138ba10f33af"
+      (reference "K?") (unit 1) (value "FINDER-34.51") (footprint "Relay_THT:Relay_SPDT_Finder_34.51_Vertical")
+    )
+    (path "/01c54577-6862-4ca7-bb55-524c2e995aee"
+      (reference "U?") (unit 1) (value "VO615A-4") (footprint "")
+    )
+    (path "/be5bbcc0-5b09-43de-a42f-297f80f602a5"
+      (reference "U?") (unit 1) (value "ESP_32") (footprint "")
+    )
+  )
 )
